File: power board 3V3 1.kicad_sch (KiCad schematic)
At the start: 20 parts, among them Q1 NMOS, Q2 PMOS, U1 TP4056-42-ESOP8, U2 HT7533-1-SOT89, U3 ${SIM.PARAMS}

Commit message: Small progress
Parts:
- added R7: 2M7, symbol Device:R
- added R8: 330k, symbol Device:R
- D3: value D_Zener -> 2V4
- R4: value R -> 330
- R5: value R -> 1M
- R6: value R -> 220k
- U3: value ${SIM.PARAMS} -> LM358DR; footprint (none) -> Package_SO:SOIC-8-1EP_3.9x4.9mm_P1.27mm_EP2.29x3mm
Connections:
- net +BATT_UVLO: now also C3.1, U2.2 (VIN)
- net Vtest: now also R7.1, R8.2; no longer R5.2, R6.1
- new net: R6.1, R7.2
- new net: R5.2, R8.1
Other:
- moved on the sheet: D3, R6, U3

Commit message: This grunt work slaps idk why people dont do more PCBs
Parts:
- added D4: 1N4148WT, Diode_SMD:D_SOD-523, symbol Diode:1N4148WT
- added Q3: PMOS - SI2301, Package_TO_SOT_SMD:SOT-23, symbol Simulation_SPICE:PMOS
- added R9: 100k, Resistor_SMD:R_0201_0603Metric, symbol Device:R
- C1, C2, C3, C4: footprint (none) -> Capacitor_SMD:C_0201_0603Metric
- D1: value LED -> LED - GREEN; footprint (none) -> LED_SMD:LED_0805_2012Metric
- D2: value LED -> LED - RED; footprint (none) -> LED_SMD:LED_0805_2012Metric
- Q1: value NMOS -> NMOS - HL3400A; footprint (none) -> Package_TO_SOT_SMD:SOT-23
- Q2: value PMOS -> PMOS - SI2301; footprint (none) -> Package_TO_SOT_SMD:SOT-23
- R1, R2: value R -> 1k; footprint (none) -> Resistor_SMD:R_0201_0603Metric
- R3, R4, R5, R6, R7, R8: footprint (none) -> Resistor_SMD:R_0201_0603Metric
Connections:
- net +5V: now also D4.2 (A), Q3.2 (G), R9.1
- net +BATT_UVLO: now also Q3.3 (S)
- net GND: now also R9.2
- new net VREG: D4.1 (K), Q3.1 (D)
Other:
- note added: "Battery + Reverse Polarity Circuit"
- note added: "Current Source Control"
- note added: "Undervoltage Lockout Circuit"
- note removed: "Reverse-polarity protection"
- note removed: "UVLO from EEE4113 Project - Gate is more negative than Source => PMOS turns on - Vopamp = A(Vref-Vtest) - If Vtest > Vref, opamp stays 0, PMOS = ON"
- moved on the sheet: C1, C2, C3, C4, D1, D2, D3, Q2, R1, R2, R3, R4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

Commit message: Almost ready to do PCB
Parts:
- added J1, J2: Conn_01x15_Pin, Connector_PinHeader_2.54mm:PinHeader_1x15_P2.54mm_Vertical, symbol Connector:Conn_01x15_Pin
- BT1: value Battery_Cell -> 18650
- D3: footprint (none) -> Diode_SMD:D_SOD-523
Connections:
- net +3V3: now also J2.11 (Pin_11); no longer C4.1, U2.3 (VOUT)
- net +5V: now also J1.13 (Pin_13), J1.4 (Pin_4); no longer C2.1, D1.2 (A), D2.2 (A), D4.2 (A), Q3.2 (G), R9.1, U1.4 (V_{CC}), U1.8 (CE)
- net +BATT: now also J1.11 (Pin_11), J1.14 (Pin_14), J1.15 (Pin_15), J1.9 (Pin_9), J2.4 (Pin_4); no longer F1.1, Q1.2 (G), Q2.3 (S), R4.1, R5.1, U1.5 (BAT), U3.3 (V+)
- net +BATT_UVLO: now also J1.3 (Pin_3), J2.1 (Pin_1); no longer C3.1, Q3.3 (S), U2.2 (VIN)
- net -BATT: now also J1.8 (Pin_8), J2.6 (Pin_6); no longer BT1.2 (-), Q1.1 (D)
- net GND: now also J2.9 (Pin_9); no longer Q1.3 (S)
- net FUSE2: now reaches BT1.1 (+), F1.2
- net FUSE2: now also J2.15 (Pin_15)
- net VREG renamed SELECTOR OUT1
- net SELECTOR OUT1: now also J1.2 (Pin_2)
- new net +BATT2: F1.1, J1.1 (Pin_1), J2.5 (Pin_5)
- new net +RPP2: J2.7 (Pin_7), Q1.2 (G)
- new net -BATT1: BT1.2 (-), J1.10 (Pin_10)
- new net -RPP2: J2.8 (Pin_8), Q1.1 (D)
- new net BATT2CHRG1: J1.12 (Pin_12), U1.5 (BAT)
- new net POW CHRGR2: C2.1, D1.2 (A), D2.2 (A), J2.3 (Pin_3), U1.4 (V_{CC}), U1.8 (CE)
- new net RPPGND1: J1.7 (Pin_7), Q1.3 (S)
- new net SELECTOR OUT2: J1.6 (Pin_6), J2.14 (Pin_14)
- new net USB2SEL2: D4.2 (A), J2.12 (Pin_12), Q3.2 (G), R9.1
- new net UVLO ON2: J2.2 (Pin_2), Q2.3 (S), R4.1, R5.1, U3.3 (V+)
- new net UVLO2SEL2: J2.13 (Pin_13), Q3.3 (S)
- new net VREG2: C3.1, J2.10 (Pin_10), U2.2 (VIN)
- new net VREGOUT1: C4.1, J1.5 (Pin_5), U2.3 (VOUT)
Other:
- note added: "- connects +BATT to charger"
- note added: "- connects +BATT to whole cct"
- note added: "- connects -BATT to whole cct"
- note added: "- connects USB input to the current selector cct"
- note added: "- connects charging cct to USBin"
- note added: "- connects regulator input"
- note added: "- connects regulator output"
- note added: "- current selector cct output"
- note added: "- rpolpro GND connection"
- note added: "- rpolpro for batt+"
- note added: "- rpolpro for batt-"
- note added: "- same but for +BATT_UVLO output"
- note added: "- short to connect UVLO cct"
- note added: "- skips uvlo and shorts it to +BATT_UVLO"
- note added: "1"
- note added: "18650 Battery Health and Regulator Module"
- note added: "Author: HARRY PAPANICOLAOU"
- note added: "Current Source Selector"
- note added: "DEBUG JUMPER PINS Left - Short Location Right - Destination"
- note removed: "Current Source Control"
- moved on the sheet: BT1, C1, C2, C3, C4, D1, D2, D3, D4, F1, Q1, Q2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

Commit message: Last footprint then pcb
Parts:
- BT1: footprint (none) -> Battery:BatteryHolder_Keystone_1042_1x18650
Changed lines of the file:
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@@
 			)
 		)
-		(property "Footprint" ""
+		(property "Footprint" "Battery:BatteryHolder_Keystone_1042_1x18650"
 			(at 22.86 34.036 90)
 			(effects

Commit message: UGH im washed
Parts:
- removed F1: 1A, symbol Device:Fuse
Changed lines of the file:
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@@
 	)
 	(junction
-		(at 22.86 21.59)
-		(diameter 0)
-		(color 0 0 0 0)
-	)
-	(junction
 		(at 17.78 127)
 		(diameter 0)
@@
 	)
 	(junction
-		(at 22.86 30.48)
-		(diameter 0)
-		(color 0 0 0 0)
-	)
-	(junction
 		(at 31.75 160.02)
 		(diameter 0)
@@
 	(wire
 		(pts
-			(xy 22.86 21.59) (xy 29.21 21.59)
-		)
-		(stroke
-			(width 0)
-			(type default)
-		)
-	)
-	(wire
-		(pts
 			(xy 21.59 165.1) (xy 21.59 166.37)
 		)
@@
 	(wire
 		(pts
-			(xy 22.86 30.48) (xy 22.86 29.21)
-		)
-		(stroke
-			(width 0)
-			(type default)
-		)
-	)
-	(wire
-		(pts
 			(xy 234.95 30.48) (xy 234.95 26.67)
 		)
@@
 	(wire
 		(pts
+			(xy 19.05 21.59) (xy 29.21 21.59)
+		)
+		(stroke
+			(width 0)
+			(type default)
+		)
+	)
+	(wire
+		(pts
 			(xy 50.8 34.29) (xy 52.07 34.29)
 		)
@@
 	(wire
 		(pts
-			(xy 19.05 21.59) (xy 22.86 21.59)
-		)
-		(stroke
-			(width 0)
-			(type default)
-		)
-	)
-	(wire
-		(pts
 			(xy 48.26 73.66) (xy 48.26 68.58)
 		)
@@
 					(unit 1)
 				)
-			)
-		)
-	)
-	(symbol
-		(lib_id "Device:Fuse")
-		(at 22.86 25.4 0)
-		(unit 1)
-		(exclude_from_sim no)
-		(in_bom yes)
-		(on_board yes)
-		(dnp no)
-		(fields_autoplaced yes)
-		(property "Reference" "F1"
-			(at 25.4 24.1299 0)
-			(effects
-				(font
-					(size 1.27 1.27)
-				)
-				(justify left)
-			)
-		)
-		(property "Value" "1A"
-			(at 25.4 26.6699 0)
-			(effects
-				(font
-					(size 1.27 1.27)
-				)
-				(justify left)
-			)
-		)
-		(property "Footprint" ""
-			(at 21.082 25.4 90)
-			(effects
-				(font
-					(size 1.27 1.27)
-				)
-				(hide yes)
-			)
-		)
-		(property "Datasheet" "~"
-			(at 22.86 25.4 0)
-			(effects
-				(font
-					(size 1.27 1.27)
-				)
-				(hide yes)
-			)
-		)
-		(property "Description" "Fuse"
-			(at 22.86 25.4 0)
-			(effects
-				(font
-					(size 1.27 1.27)
-				)
-				(hide yes)
-			)
-		)
-		(pin "1"
-		)
-		(pin "2"
-		)
-		(instances
-			(project ""
-				(path "/fab2136b-e420-428a-99c6-bb02c3ef62e3"
-					(reference "F1")
-					(unit 1)
-				)

Commit message: Ugh
Parts:
- removed J1, J2: Conn_01x15_Pin, Connector_PinHeader_2.54mm:PinHeader_1x15_P2.54mm_Vertical, symbol Connector:Conn_01x15_Pin
- added J1: Conn_02x15_Odd_Even, Connector_PinHeader_2.54mm:PinHeader_2x15_P2.54mm_Vertical, symbol Connector_Generic:Conn_02x15_Odd_Even
Connections:
- net +3V3: now also J1.22 (Pin_22)
- net +5V: now also J1.23 (Pin_23), J1.5 (Pin_5)
- net +BATT: now also J1.1 (Pin_1), J1.13 (Pin_13), J1.3 (Pin_3), J1.8 (Pin_8), J1.9 (Pin_9)
- net +BATT2: now also J1.10 (Pin_10), J1.29 (Pin_29)
- net +BATT_UVLO: now also J1.2 (Pin_2), J1.25 (Pin_25)
- net +RPP2: now also J1.14 (Pin_14)
- net -BATT: now also J1.12 (Pin_12), J1.15 (Pin_15)
- net -BATT1: now also J1.11 (Pin_11)
- net -RPP2: now also J1.16 (Pin_16)
- net BATT2CHRG1: now also J1.7 (Pin_7)
- net FUSE2: now also J1.30 (Pin_30)
- net GND: now also J1.18 (Pin_18)
- net POW CHRGR2: now also J1.6 (Pin_6)
- net RPPGND1: now also J1.17 (Pin_17)
- net SELECTOR OUT1: now also J1.27 (Pin_27)
- net SELECTOR OUT2: now also J1.19 (Pin_19), J1.28 (Pin_28)
- net USB2SEL2: now also J1.24 (Pin_24)
- net UVLO ON2: now also J1.4 (Pin_4)
- net UVLO2SEL2: now also J1.26 (Pin_26)
- net VREG2: now also J1.20 (Pin_20)
- net VREGOUT1: now also J1.21 (Pin_21)
Changed lines of the file:
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@@
 	)
 	(label "UVLO ON2"
-		(at 212.09 91.44 0)
+		(at 210.82 91.44 0)
 		(effects
 			(font
@@
 	)
 	(label "+RPP2"
-		(at 212.09 104.14 0)
+		(at 210.82 104.14 0)
 		(effects
 			(font
@@
 	)
 	(label "SELECTOR OUT2"
-		(at 212.09 121.92 0)
+		(at 210.82 121.92 0)
 		(effects
 			(font
@@
 	)
 	(label "-BATT2"
-		(at 212.09 101.6 0)
+		(at 210.82 101.6 0)
 		(effects
 			(font
@@
 	)
 	(label "VREGOUT2"
-		(at 212.09 114.3 0)
+		(at 210.82 114.3 0)
 		(effects
 			(font
@@
 	)
 	(label "USB2SEL2"
-		(at 212.09 116.84 0)
+		(at 210.82 116.84 0)
 		(effects
 			(font
@@
 	)
 	(label "+BATT_UVLO"
-		(at 212.09 88.9 0)
+		(at 210.82 88.9 0)
 		(effects
 			(font
@@
 	)
 	(label "+BATT2"
-		(at 212.09 99.06 0)
+		(at 210.82 99.06 0)
 		(effects
 			(font
@@
 	)
 	(label "BATT2CHRG2"
-		(at 212.09 96.52 0)
+		(at 210.82 96.52 0)
 		(effects
 			(font
@@
 	)
 	(label "FUSE2"
-		(at 212.09 124.46 0)
+		(at 210.82 124.46 0)
 		(effects
 			(font
@@
 	)
 	(label "UVLO2SEL2"
-		(at 212.09 119.38 0)
+		(at 210.82 119.38 0)
 		(effects
 			(font
@@
 	)
 	(label "-RPP2"
-		(at 212.09 106.68 0)
+		(at 210.82 106.68 0)
 		(effects
 			(font
@@
 	)
 	(label "VREG2"
-		(at 212.09 111.76 0)
+		(at 210.82 111.76 0)
 		(effects
 			(font
@@
 	)
 	(label "POW CHRGR2"
-		(at 212.09 93.98 0)
+		(at 210.82 93.98 0)
 		(effects
 			(font
@@
 	)
 	(label "RPPGND2"
-		(at 212.09 109.22 0)
+		(at 210.82 109.22 0)
 		(effects
 			(font
@@
 	)
 	(symbol
-		(lib_id "Connector:Conn_01x15_Pin")
-		(at 207.01 106.68 0)
-		(unit 1)
-		(exclude_from_sim no)
-		(in_bom yes)
-		(on_board yes)
-		(dnp no)
-		(property "Reference" "J2"
-			(at 216.154 83.312 0)
-			(effects
-				(font
-					(size 1.27 1.27)
-				)
-				(justify right)
-			)
-		)
-		(property "Value" "Conn_01x15_Pin"
-			(at 223.52 85.344 0)
-			(effects
-				(font
-					(size 1.27 1.27)
-				)
-				(justify right)
-			)
-		)
-		(property "Footprint" "Connector_PinHeader_2.54mm:PinHeader_1x15_P2.54mm_Vertical"
-			(at 207.01 106.68 0)
-			(effects
-				(font
-					(size 1.27 1.27)
-				)
-				(hide yes)
-			)
-		)
-		(property "Datasheet" "~"
-			(at 207.01 106.68 0)
-			(effects
-				(font
-					(size 1.27 1.27)
-				)
-				(hide yes)
-			)
-		)
-		(property "Description" "Generic connector, single row, 01x15, script generated"
-			(at 207.01 106.68 0)
-			(effects
-				(font
-					(size 1.27 1.27)
-				)
-				(hide yes)
-			)
-		)
-		(pin "1"
-		)
-		(pin "3"
-		)
-		(pin "10"
-		)
-		(pin "15"
-		)
-		(pin "14"
-		)
-		(pin "2"
-		)
-		(pin "9"
-		)
-		(pin "5"
-		)
-		(pin "13"
-		)
-		(pin "6"
-		)
-		(pin "12"
-		)
-		(pin "8"
-		)
-		(pin "11"
-		)
-		(pin "4"
-		)
-		(pin "7"
-		)
-		(instances
-			(project "power board 3V3 1"
-				(path "/fab2136b-e420-428a-99c6-bb02c3ef62e3"
-					(reference "J2")
-					(unit 1)
-				)
-			)
-		)
-	)
-	(symbol
 		(lib_id "power:GND")
 		(at 31.75 189.23 0)
@@
 	)
 	(symbol
-		(lib_id "Connector:Conn_01x15_Pin")
-		(at 203.2 106.68 180)
-		(unit 1)
-		(exclude_from_sim no)
-		(in_bom yes)
-		(on_board yes)
-		(dnp no)
-		(property "Reference" "J1"
-			(at 187.452 82.804 0)
-			(effects
-				(font
-					(size 1.27 1.27)
-				)
-				(justify right)
-			)
-		)
-		(property "Value" "Conn_01x15_Pin"
-			(at 187.452 85.344 0)
-			(effects
-				(font
-					(size 1.27 1.27)
-				)
-				(justify right)
-			)
-		)
-		(property "Footprint" "Connector_PinHeader_2.54mm:PinHeader_1x15_P2.54mm_Vertical"
-			(at 203.2 106.68 0)
-			(effects
-				(font
-					(size 1.27 1.27)
-				)
-				(hide yes)
-			)
-		)
-		(property "Datasheet" "~"
-			(at 203.2 106.68 0)
-			(effects
-				(font
-					(size 1.27 1.27)
-				)
-				(hide yes)
-			)
-		)
-		(property "Description" "Generic connector, single row, 01x15, script generated"
-			(at 203.2 106.68 0)
-			(effects
-				(font
-					(size 1.27 1.27)
-				)
-				(hide yes)
-			)
-		)
-		(pin "1"
-		)
-		(pin "3"
-		)
-		(pin "10"
-		)
-		(pin "15"
-		)
-		(pin "14"
-		)
-		(pin "2"
-		)
-		(pin "9"
-		)
-		(pin "5"
-		)
-		(pin "13"
-		)
-		(pin "6"
-		)
-		(pin "12"
-		)
-		(pin "8"
-		)
-		(pin "11"
-		)
-		(pin "4"
-		)
-		(pin "7"
-		)
-		(instances
-			(project ""
-				(path "/fab2136b-e420-428a-99c6-bb02c3ef62e3"
-					(reference "J1")
-					(unit 1)
-				)
-			)
-		)
-	)
-	(symbol
 		(lib_id "Simulation_SPICE:PMOS")
 		(at 125.73 43.18 270)
@@
 					(unit 1)
 				)
+			)
+		)
+	)
+	(symbol
+		(lib_id "Connector_Generic:Conn_02x15_Odd_Even")
+		(at 203.2 106.68 0)
+		(unit 1)
+		(exclude_from_sim no)
+		(in_bom yes)
+		(on_board yes)
+		(dnp no)
+		(fields_autoplaced yes)
+		(property "Reference" "J1"
+			(at 204.47 82.55 0)
+			(effects
+				(font
+					(size 1.27 1.27)
+				)
+			)
+		)
+		(property "Value" "Conn_02x15_Odd_Even"
+			(at 204.47 85.09 0)
+			(effects
+				(font
+					(size 1.27 1.27)
+				)
+			)
+		)
+		(property "Footprint" "Connector_PinHeader_2.54mm:PinHeader_2x15_P2.54mm_Vertical"
+			(at 203.2 106.68 0)
+			(effects
+				(font
+					(size 1.27 1.27)
+				)
+				(hide yes)
+			)
+		)
+		(property "Datasheet" "~"
+			(at 203.2 106.68 0)
+			(effects
+				(font
+					(size 1.27 1.27)
+				)
+				(hide yes)
+			)
+		)
+		(property "Description" "Generic connector, double row, 02x15, odd/even pin numbering scheme (row 1 odd numbers, row 2 even numbers), script generated (kicad-library-utils/schlib/autogen/connector/)"
+			(at 203.2 106.68 0)
+			(effects
+				(font
+					(size 1.27 1.27)
+				)
+				(hide yes)
+			)
+		)
+		(pin "7"
+		)
+		(pin "11"
+		)
+		(pin "8"
+		)
+		(pin "26"
+		)
+		(pin "15"
+		)
+		(pin "14"
+		)
+		(pin "17"
+		)
+		(pin "19"
+		)
+		(pin "16"
+		)
+		(pin "18"
+		)
+		(pin "10"
+		)
+		(pin "13"
+		)
+		(pin "29"
+		)
+		(pin "1"
+		)
+		(pin "3"
+		)
+		(pin "24"
+		)
+		(pin "6"
+		)
+		(pin "2"
+		)
+		(pin "27"
+		)
+		(pin "9"
+		)
+		(pin "21"
+		)
+		(pin "20"
+		)
+		(pin "28"
+		)
+		(pin "22"
+		)
+		(pin "23"
+		)
+		(pin "5"
+		)
+		(pin "4"
+		)
+		(pin "12"
+		)
+		(pin "25"
+		)
+		(pin "30"
+		)
+		(instances
+			(project ""
+				(path "/fab2136b-e420-428a-99c6-bb02c3ef62e3"
+					(reference "J1")
+					(unit 1)
+				)

Commit message: Next is just silk screen labelling and ask Si Teng if Im retarded
Parts:
- removed J1: Conn_02x15_Odd_Even, Connector_PinHeader_2.54mm:PinHeader_2x15_P2.54mm_Vertical, symbol Connector_Generic:Conn_02x15_Odd_Even
- added J1: Conn_02x14_Odd_Even, Connector_PinHeader_2.54mm:PinHeader_2x14_P2.54mm_Vertical, symbol Connector_Generic:Conn_02x14_Odd_Even
Connections:
- net FUSE2 is gone; now on net +BATT2: BT1.1 (+)
- net +3V3: now also J1.24 (Pin_24)
- net +5V: now also J1.17 (Pin_17), J1.9 (Pin_9)
- net +BATT: now also J1.1 (Pin_1), J1.11 (Pin_11), J1.13 (Pin_13), J1.3 (Pin_3), J1.8 (Pin_8)
- net +BATT2: now also J1.2 (Pin_2)
- net +BATT_UVLO: now also J1.12 (Pin_12), J1.15 (Pin_15)
- net +RPP2: now also J1.4 (Pin_4)
- net -BATT: now also J1.25 (Pin_25), J1.28 (Pin_28)
- net -BATT1: now also J1.27 (Pin_27)
- net -RPP2: now also J1.26 (Pin_26)
- net BATT2CHRG1: now also J1.7 (Pin_7)
- net GND: now also J1.6 (Pin_6)
- net POW CHRGR2: now also J1.10 (Pin_10)
- net RPPGND1: now also J1.5 (Pin_5)
- net SELECTOR OUT1: now also J1.19 (Pin_19)
- net SELECTOR OUT2: now also J1.20 (Pin_20), J1.21 (Pin_21)
- net USB2SEL2: now also J1.18 (Pin_18)
- net UVLO ON2: now also J1.14 (Pin_14)
- net UVLO2SEL2: now also J1.16 (Pin_16)
- net VREG2: now also J1.22 (Pin_22)
- net VREGOUT1: now also J1.23 (Pin_23)
Other:
- note added: "DEBUG JUMPER PINS"
- note removed: "- connects +BATT to charger"
- note removed: "- connects +BATT to whole cct"
- note removed: "- connects -BATT to whole cct"
- note removed: "- connects USB input to the current selector cct"
- note removed: "- connects charging cct to USBin"
- note removed: "- connects regulator input"
- note removed: "- connects regulator output"
- note removed: "- current selector cct output"
- note removed: "- rpolpro GND connection"
- note removed: "- rpolpro for batt+"
- note removed: "- rpolpro for batt-"
- note removed: "- same but for +BATT_UVLO output"
- note removed: "- short to connect UVLO cct"
- note removed: "- skips uvlo and shorts it to +BATT_UVLO"
- note removed: "DEBUG JUMPER PINS Left - Short Location Right - Destination"
