File: power board 3V3 1.kicad_sch (KiCad schematic)
At the start: 29 parts, among them J1 UVLO TP, J2 CHRGR TP, J3 BATT & RPP TP, J4 LDO TP, J5 SRC CTRL TP, Q1 NMOS - HL3400A, Q2 PMOS - SI2301, Q3 PMOS - SI2301, U1 TP4056-42-ESOP8, U2 HT7533-1-SOT89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

Commit message: PCB looks better now
Parts:
- BT1: footprint Battery:BatteryHolder_Keystone_1042_1x18650 -> Connector_PinHeader_2.54mm:PinHeader_1x02_P2.54mm_Vertical; now not fitted
Connections:
- net POW CHRGR2 is gone; now on net +5V: C2.1, D1.2 (A), D2.2 (A), J2.2 (Pin_2), U1.4 (V_{CC}), U1.8 (CE)
Changed lines of the file:
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@@
 	)
 	(junction
+		(at 48.26 73.66)
+		(diameter 0)
+		(color 0 0 0 0)
+	)
+	(junction
 		(at 74.93 107.95)
 		(diameter 0)
@@
 	)
 	(junction
+		(at 48.26 69.85)
+		(diameter 0)
+		(color 0 0 0 0)
+	)
+	(junction
 		(at 203.2 90.17)
 		(diameter 0)
@@
 	(wire
 		(pts
+			(xy 48.26 69.85) (xy 48.26 73.66)
+		)
+		(stroke
+			(width 0)
+			(type default)
+		)
+	)
+	(wire
+		(pts
 			(xy 74.93 102.87) (xy 74.93 107.95)
 		)
@@
 		(in_bom yes)
 		(on_board yes)
-		(dnp no)
+		(dnp yes)
 		(fields_autoplaced yes)
 		(property "Reference" "BT1"
@@
 			)
 		)
-		(property "Footprint" "Battery:BatteryHolder_Keystone_1042_1x18650"
+		(property "Footprint" "Connector_PinHeader_2.54mm:PinHeader_1x02_P2.54mm_Vertical"
 			(at 22.86 34.036 90)
 			(effects
